File: music_box.sch (KiCad schematic (older format))
At the start: 39 parts, among them J1 USB_C_Receptacle, J2 UART, P1 ICSPforPICKit, Q1 IRLML6402, Q2 IRLML6402, SW1 SW_Push, U1 CH340E, U2 PIC16(L)F18324, U3 24FC256, U4 TC118SS, U5 TLV61225

Commit message: ver2
Parts:
- removed C2: 0.1u, Capacitor_SMD:C_0603_1608Metric_Pad1.05x0.95mm_HandSolder, symbol Device:C
- removed D1: GS1010FL, Diode_SMD:D_SOD-123F, symbol Device:D
- removed D2: RB751S-40, Diode_SMD:D_SOD-523, symbol Device:D
- removed J2: UART, Connector_PinHeader_2.54mm:PinHeader_1x04_P2.54mm_Vertical, symbol Connector:Conn_01x04_Female
- removed JP2: D1_Bridge, Jumper:SolderJumper-2_P1.3mm_Open_RoundedPad1.0x1.5mm, symbol Jumper:SolderJumper_2_Open
- removed JP3: SP_SORCE, Jumper:SolderJumper-3_P1.3mm_Open_RoundedPad1.0x1.5mm_NumberLabels, symbol Jumper:SolderJumper_3_Open
- removed L1: L, Inductor_THT:L_Axial_L9.5mm_D4.0mm_P12.70mm_Horizontal_Fastron_SMCC, symbol Device:L
- removed Q1, Q2: IRLML6402, Package_TO_SOT_SMD:SOT-23, symbol fues-device:MOS_P_ENHANCE_GSD
- removed R6: 5.1k, Resistor_SMD:R_0603_1608Metric_Pad1.05x0.95mm_HandSolder, symbol Device:R
- removed U5: TLV61225, Package_TO_SOT_SMD:SOT-363_SC-70-6, symbol fues-IC_and_module:TLV61225
- added D1: RB411D, Package_TO_SOT_SMD:SC-59, symbol Device:D_Schottky_AAK
- added D2: LED NC, Diode_SMD:D_0603_1608Metric_Pad1.05x0.95mm_HandSolder, symbol Device:LED
- added L1: 100uH, Inductor_THT:L_Axial_L9.5mm_D4.0mm_P12.70mm_Horizontal_Fastron_SMCC, symbol Device:L_Small
- added Q1, Q2: 2n7002, Package_TO_SOT_SMD:SOT-23, symbol Device:Q_NMOS_GSD
- added R1, R10, R11, R2, R3, R4: 10k, Resistor_SMD:R_0603_1608Metric_Pad1.05x0.95mm_HandSolder, symbol Device:R
- added R14, R15: 47, Resistor_SMD:R_0603_1608Metric_Pad1.05x0.95mm_HandSolder, symbol Device:R
- added SW1: POWER, fues-connect:2.54-2pin-lay, symbol Switch:SW_SPST
- added TP1: tp_PC2MC, TestPoint:TestPoint_Pad_D2.0mm, symbol Connector:TestPoint_Flag
- added TP2: tp_MC2PC, TestPoint:TestPoint_Pad_D2.0mm, symbol Connector:TestPoint_Flag
- added TP3: tp_GND, TestPoint:TestPoint_Pad_D2.0mm, symbol Connector:TestPoint_Flag
- added U1: HT77XXA_SOT-25, Package_TO_SOT_SMD:TSOT-23-5, symbol fues-IC_and_module:HT77XXA_SOT-25
- C1: renamed from C7; value C -> 47u; footprint Capacitor_SMD:C_0805_2012Metric_Pad1.15x1.40mm_HandSolder -> Capacitor_SMD:C_1210_3225Metric_Pad1.42x2.65mm_HandSolder
- C2: renamed from C8; value C -> 22u; footprint Capacitor_SMD:C_0805_2012Metric_Pad1.15x1.40mm_HandSolder -> Capacitor_SMD:C_0603_1608Metric_Pad1.05x0.95mm_HandSolder
- C3: renamed from C1; value 0.1u -> 0.1u 1608
- C4: renamed from C3; value 0.1u -> 0.1u 1608
- C5: value 0.1u -> 0.1u 1608
- C6: renamed from C4; value 0.1u -> 0.1u 1608
- C7: renamed from C6; value 0.1u -> 0.1u 1608
- H1, H2, H3, H4: footprint fues-mounting_hole:M2-drillHole -> fues-mounting_hole:M2-drillHole_nosilk_nopad
- R7: value 5.1k -> 470 NC
- SP1: value buzzer -> sp; symbol Device:Speaker_Crystal -> Device:Speaker
- renumbered BT2 to BT1, BT1 to BT2, R2 to R12, R3 to R13, R1 to R5, R8 to R6, R4 to R8, R5 to R9, SW1 to SW2, U1 to U2, U2 to U3, U3 to U4, U4 to U5
Connections:
- net VDD is gone; now on net +3V3: C5.1, C6.1, P1.2 (VDD), R12.1, R13.1, U3.1 (VDD), U4.8 (VCC)
- net +3V3: now also D1.3 (K), U1.1 (CE), U1.2 (VOUT)
- net +5V: now also R5.1
- net +BATT: now also C7.1, U5.4 (VDD), L1.1, R10.1, R11.1, SW1.2 (B); no longer BT1.1 (+)
- net GND: now also D2.1 (K), Q1.2 (S), Q2.2 (S), R1.2, R2.2, R3.2, R4.2, TP3.1, U1.4 (GND); no longer R7.2
- net SPD1: now also Q1.1 (G); no longer U5.2 (INA)
- net SPD2: now also Q2.1 (G); no longer U5.3 (INB)
- net UART_MC2PC: now also TP2.1
- net UART_PC2MC: now also TP1.1
- net FLOATING: now reaches U3.11 (RA2)
- net at SP1.1: now also R14.2, R15.2; no longer U5.8 (OUTA)
- net at J1.A5 (CC1): now also R3.1, R4.1; no longer R7.1
- net at J1.B5 (CC2): now also R1.1, R2.1
- net at U2.6 (TNOW): now also R7.1
- new net: R14.1, R15.1, U5.8 (OUTA)
- new net: BT1.1 (+), SW1.1 (A)
- new net: D2.2 (A), R7.2
- new net: D1.1 (A), D1.2 (A), L1.2, U1.5 (LX)
- new net SPD1_1: Q1.3 (D), R10.2, U5.2 (INA)
- new net SPD2_1: Q2.3 (D), R11.2, U5.3 (INB)
- no-connect marks 13 -> 11
Other:
- moved on the sheet: BT1, BT2, C1, C2, C3, C4, C5, C6, C7, H1, H2, H3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
